Commit message: rviz->gazebo

File: install/engineer_description/share/engineer_description/urdf/engineer_total.urdf (robot description, URDF)
Before this commit: robot engineer_total, 14 links, 13 joints
Joints:
- joint J4_joint: limit lower=0 upper=0 effort=0 velocity=0 -> lower=-5 upper=5 effort=0 velocity=0
- joint J5_joint: limit lower=0 upper=0 effort=0 velocity=0 -> lower=-5 upper=5 effort=0 velocity=0
- joint J6_joint: limit lower=0 upper=0 effort=0 velocity=0 -> lower=-5 upper=5 effort=0 velocity=0
- joint Wheel_r_b_joint: axis 0 0 0 -> 0 0 1; type fixed -> continuous
